File: ATM8_mainboard.brd (EAGLE design)
At the start: 114.3 x 60.6 mm, 44 parts, among them IC1_POSUV MEGA8-P, IC2_VRETENO MEGA8-P, J1 22-27-2021-02, J2 22-27-2021-02

Commit message: 
Parts:
- moved SV2 32.7 mm to (20.3, 14.0), turned to 0 degrees
- moved LPT1 16.5 mm to (57.1, 14.0), turned to 90 degrees
- moved R13 15.7 mm to (54.6, 38.1), turned to 270 degrees
- moved Q2 11.7 mm to (41.9, 17.8), turned to 90 degrees
- moved R18 10.8 mm to (77.5, 52.1), turned to 0 degrees
- moved R7 10.2 mm to (48.3, 17.8), turned to 270 degrees
- moved Q1 10.2 mm to (96.5, 19.1)
- moved LPT2 9.25 mm to (64.8, 44.5), turned to 0 degrees
- moved R17 8.52 mm to (74.9, 49.5), turned to 0 degrees
- moved R8 8.13 mm to (74.9, 10.2), turned to 180 degrees
- moved INPUTCNC 8.03 mm to (67.3, 57.1), turned to 180 degrees
- moved R12 8.03 mm to (53.3, 20.3), turned to 270 degrees
- moved J1 6.48 mm to (86.4, 8.89), turned to 180 degrees
- moved R9 6.35 mm to (72.4, 12.7), turned to 180 degrees
- moved R10 5.24 mm to (69.8, 15.2), turned to 180 degrees
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Routing:
- net GND: track 0.00 -> 242.3 mm
- net VCC: track 0.00 -> 148.3 mm
- net ENABLE: track 0.00 -> 91.9 mm
- net RESET2: track 0.00 -> 77.2 mm
- net MOSI1: track 0.00 -> 44.5 mm
- net MISO1: track 0.00 -> 43.2 mm
- net PD41: track 0.00 -> 35.3 mm
- net PB7: track 0.00 -> 31.1 mm
- net SCL1: track 0.00 -> 22.9 mm
- net SDA1: track 0.00 -> 22.4 mm
- net PD52: track 0.00 -> 21.9 mm
- net SCK2: track 0.00 -> 20.9 mm
- net I: track 0.00 -> 20.3 mm
- net V: track 0.00 -> 17.8 mm
- net DORX: track 0.00 -> 17.8 mm
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